File: autko.kicad_sch (KiCad schematic)
At the start: 0 parts

Commit message: Initial microcontroller schematic
Other:
- sheet Microcontroller ports: added SENSOR[1..7]; removed SENSORS[1..7]
Changed lines of the file:
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@@
       (effects (font (size 1.27 1.27)) (justify left top) hide)
-    )
-    (pin "SENSORS[1..7]" input (at 46.99 43.18 180)
-      (effects (font (size 1.27 1.27)) (justify left))
     )
     (pin "IR_LEDS_ON" output (at 46.99 40.64 180)
@@
       (effects (font (size 1.27 1.27)) (justify right))
     )
+    (pin "SENSOR[1..7]" input (at 46.99 43.18 180)
+      (effects (font (size 1.27 1.27)) (justify left))
+    )
     (instances
