File: Bluetooth.kicad_sch (KiCad schematic)
At the start: 0 parts

Commit message: Bluetooth initial schematic
Parts:
- added C?: 10uF, symbol Device:C
- added C?: 100nF, symbol Device:C
- added D?: LED, symbol Device:LED
- added JP? (x3): Jumper_2_Bridged, symbol Jumper:Jumper_2_Bridged
- added Q?: BC807, Package_TO_SOT_SMD:SOT-23, symbol Transistor_BJT:BC807
- added R?: ?R, symbol Device:R
- added R?: 4.7kR, symbol Device:R
- added R? (x2): 10kR, symbol Device:R
- added U?: RN4870, symbol Autko:RN4870
Connections:
- new net: Q?.3 (C), R?.1
- new net: D?.2 (A), R?.2
- new net: Q?.1 (B), R?.2
- new net: JP?.1 (A), U?.23 (UART_TX)
- new net: JP?.1 (A), U?.22 (UART_RX)
- new net +3.3V: C?.1, JP?.2 (B), Q?.2 (E), R?.1, U?.4 (VBAT)
- new net GND: C?.2, C?.2, D?.1 (K), R?.2, U?.1 (GND), U?.2 (GND), U?.3 (GND), U?.31 (GND), U?.32 (GND), U?.33 (GND)
- new net LED: R?.1, U?.30 (P0_2/LED0)
- new net MODE: JP?.1 (A), R?.1, U?.18 (P2_0)
- new net ~{RST}: C?.1, R?.2, U?.21 (~{RST})
- no-connect marks 0 -> 17

Commit message: Bluetooth schematic
Parts:
- removed JP?: Jumper_2_Bridged, symbol Jumper:Jumper_2_Bridged
- removed R?: 10kR, symbol Device:R
- added C? (x2): 100nF, symbol Device:C
- added JP?: RUN/CONFIG, symbol Jumper:Jumper_2_Bridged
- added R?: 10kR, symbol Device:R
- added U?: TXB0102DCU, Package_SO:VSSOP-8_2.4x2.1mm_P0.5mm, symbol Logic_LevelTranslator:TXB0102DCU
- D?: value LED -> BLUE
Connections:
- net +3.3V: now also C?.2, JP?.1 (A), R?.2, U?.3 (VCCA), U?.6 (OE)
- net GND: now also C?.1, C?.2, U?.2 (GND)
- net RX: now also U?.1 (B2)
- net TX: now also U?.8 (B1)
- net at JP?.2 (B): now also U?.5 (A1)
- net at JP?.2 (B): now also U?.4 (A2)
- net LED: no longer names the net of R?.1, U?.30 (P0_2/LED0)
- net MODE: no longer names the net of R?.1, U?.18 (P2_0)
- net MODE: now also JP?.2 (B)
- net ~{RST}: no longer names the net of C?.1, U?.21 (~{RST})
- net ~{RST}: now also R?.1
- new net +5V: C?.1, U?.7 (VCCB)
Other:
- note added: "Bluetooth"
- note added: "Logic level converter"
- moved on the sheet: C?, D?, JP?, Q?, R?, U?

Commit message: Annotate schematics
Parts:
- gave numbers to parts that had none: 15

Commit message: ERC fixes
Connections:
- no-connect marks 17 -> 16
Changed lines of the file:
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@@
   (no_connect (at 49.53 85.09))
   (no_connect (at 80.01 53.34))
-  (no_connect (at 62.23 85.09))
   (no_connect (at 34.29 68.58))
   (no_connect (at 52.07 85.09))
