File: pcb/Motors.kicad_sch (KiCad schematic)
At the start: 11 parts, among them M1 LEFT, M2 RIGHT, U12 TB6612FNG

Commit message: Power switch footprint and initial pcb
Parts:
- renumbered U12 to U11
Changed lines of the file:
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@@
   (symbol (lib_id "power:+3.3V") (at 46.99 58.42 0) (unit 1)
     (in_bom yes) (on_board yes) (dnp no) (fields_autoplaced)
-    (property "Reference" "#PWR043" (at 46.99 62.23 0)
+    (property "Reference" "#PWR042" (at 46.99 62.23 0)
       (effects (font (size 1.27 1.27)) hide)
     )
@@
       (project "Autko"
         (path "/8d5cfdec-de34-4148-9100-7125640c46f5/541574ca-21e4-445f-b8e2-ded2c59d3b8a"
-          (reference "#PWR043") (unit 1)
+          (reference "#PWR042") (unit 1)
         )
       )
@@
   (symbol (lib_id "Driver_Motor:TB6612FNG") (at 64.77 69.85 0) (unit 1)
     (in_bom yes) (on_board yes) (dnp no) (fields_autoplaced)
-    (property "Reference" "U12" (at 74.3459 92.71 0)
+    (property "Reference" "U11" (at 74.3459 92.71 0)
       (effects (font (size 1.27 1.27)) (justify left))
     )
@@
       (project "Autko"
         (path "/8d5cfdec-de34-4148-9100-7125640c46f5/541574ca-21e4-445f-b8e2-ded2c59d3b8a"
-          (reference "U12") (unit 1)
+          (reference "U11") (unit 1)
         )
       )
@@
   (symbol (lib_id "power:GND") (at 90.17 44.45 0) (unit 1)
     (in_bom yes) (on_board yes) (dnp no)
-    (property "Reference" "#PWR042" (at 90.17 50.8 0)
+    (property "Reference" "#PWR041" (at 90.17 50.8 0)
       (effects (font (size 1.27 1.27)) hide)
     )
@@
       (project "Autko"
         (path "/8d5cfdec-de34-4148-9100-7125640c46f5/541574ca-21e4-445f-b8e2-ded2c59d3b8a"
-          (reference "#PWR042") (unit 1)
+          (reference "#PWR041") (unit 1)
         )
       )
@@
   (symbol (lib_id "power:+3.3V") (at 34.29 31.75 0) (unit 1)
     (in_bom yes) (on_board yes) (dnp no) (fields_autoplaced)
-    (property "Reference" "#PWR039" (at 34.29 35.56 0)
+    (property "Reference" "#PWR038" (at 34.29 35.56 0)
       (effects (font (size 1.27 1.27)) hide)
     )
@@
       (project "Autko"
         (path "/8d5cfdec-de34-4148-9100-7125640c46f5/541574ca-21e4-445f-b8e2-ded2c59d3b8a"
-          (reference "#PWR039") (unit 1)
+          (reference "#PWR038") (unit 1)
         )
       )
@@
   (symbol (lib_id "power:+7.5V") (at 90.17 31.75 0) (unit 1)
     (in_bom yes) (on_board yes) (dnp no) (fields_autoplaced)
-    (property "Reference" "#PWR040" (at 90.17 35.56 0)
+    (property "Reference" "#PWR039" (at 90.17 35.56 0)
       (effects (font (size 1.27 1.27)) hide)
     )
@@
       (project "Autko"
         (path "/8d5cfdec-de34-4148-9100-7125640c46f5/541574ca-21e4-445f-b8e2-ded2c59d3b8a"
+          (reference "#PWR039") (unit 1)
+        )
+      )
+    )
+  )
+  (symbol (lib_id "Device:C_Polarized") (at 34.29 38.1 0) (unit 1)
+    (in_bom yes) (on_board yes) (dnp no)
+    (property "Reference" "C20" (at 36.83 36.83 0)
+      (effects (font (size 1.27 1.27)) (justify left))
+    )
+    (property "Value" "10uF" (at 36.83 39.37 0)
+      (effects (font (size 1.27 1.27)) (justify left))
+    )
+    (property "Footprint" "Capacitor_Tantalum_SMD:CP_EIA-3216-18_Kemet-A" (at 35.2552 41.91 0)
+      (effects (font (size 1.27 1.27)) hide)
+    )
+    (property "Datasheet" "~" (at 34.29 38.1 0)
+      (effects (font (size 1.27 1.27)) hide)
+    )
+    (pin "1")
+    (pin "2")
+    (instances
+      (project "Autko"
+        (path "/8d5cfdec-de34-4148-9100-7125640c46f5/541574ca-21e4-445f-b8e2-ded2c59d3b8a"
+          (reference "C20") (unit 1)
+        )
+      )
+    )
+  )
+  (symbol (lib_id "Device:C") (at 92.71 59.69 0) (mirror y) (unit 1)
+    (in_bom yes) (on_board yes) (dnp no)
+    (property "Reference" "C24" (at 90.17 58.42 0)
+      (effects (font (size 1.27 1.27)) (justify left))
+    )
+    (property "Value" "100nF" (at 90.17 60.96 0)
+      (effects (font (size 1.27 1.27)) (justify left))
+    )
+    (property "Footprint" "Capacitor_SMD:C_0805_2012Metric" (at 91.7448 63.5 0)
+      (effects (font (size 1.27 1.27)) hide)
+    )
+    (property "Datasheet" "~" (at 92.71 59.69 0)
+      (effects (font (size 1.27 1.27)) hide)
+    )
+    (pin "1")
+    (pin "2")
+    (instances
+      (project "Autko"
+        (path "/8d5cfdec-de34-4148-9100-7125640c46f5/541574ca-21e4-445f-b8e2-ded2c59d3b8a"
+          (reference "C24") (unit 1)
+        )
+      )
+    )
+  )
+  (symbol (lib_id "Device:C") (at 77.47 38.1 0) (unit 1)
+    (in_bom yes) (on_board yes) (dnp no)
+    (property "Reference" "C22" (at 80.01 36.83 0)
+      (effects (font (size 1.27 1.27)) (justify left))
+    )
+    (property "Value" "100nF" (at 80.01 39.37 0)
+      (effects (font (size 1.27 1.27)) (justify left))
+    )
+    (property "Footprint" "Capacitor_SMD:C_0805_2012Metric" (at 78.4352 41.91 0)
+      (effects (font (size 1.27 1.27)) hide)
+    )
+    (property "Datasheet" "~" (at 77.47 38.1 0)
+      (effects (font (size 1.27 1.27)) hide)
+    )
+    (pin "1")
+    (pin "2")
+    (instances
+      (project "Autko"
+        (path "/8d5cfdec-de34-4148-9100-7125640c46f5/541574ca-21e4-445f-b8e2-ded2c59d3b8a"
+          (reference "C22") (unit 1)
+        )
+      )
+    )
+  )
+  (symbol (lib_id "power:GND") (at 34.29 44.45 0) (unit 1)
+    (in_bom yes) (on_board yes) (dnp no)
+    (property "Reference" "#PWR040" (at 34.29 50.8 0)
+      (effects (font (size 1.27 1.27)) hide)
+    )
+    (property "Value" "GND" (at 34.29 48.26 0)
+      (effects (font (size 1.27 1.27)))
+    )
+    (property "Footprint" "" (at 34.29 44.45 0)
+      (effects (font (size 1.27 1.27)) hide)
+    )
+    (property "Datasheet" "" (at 34.29 44.45 0)
+      (effects (font (size 1.27 1.27)) hide)
+    )
+    (pin "1")
+    (instances
+      (project "Autko"
+        (path "/8d5cfdec-de34-4148-9100-7125640c46f5/541574ca-21e4-445f-b8e2-ded2c59d3b8a"
           (reference "#PWR040") (unit 1)
         )
@@
     )
   )
-  (symbol (lib_id "Device:C_Polarized") (at 34.29 38.1 0) (unit 1)
-    (in_bom yes) (on_board yes) (dnp no)
-    (property "Reference" "C20" (at 36.83 36.83 0)
-      (effects (font (size 1.27 1.27)) (justify left))
-    )
-    (property "Value" "10uF" (at 36.83 39.37 0)
-      (effects (font (size 1.27 1.27)) (justify left))
-    )
-    (property "Footprint" "Capacitor_Tantalum_SMD:CP_EIA-3216-18_Kemet-A" (at 35.2552 41.91 0)
-      (effects (font (size 1.27 1.27)) hide)
-    )
-    (property "Datasheet" "~" (at 34.29 38.1 0)
-      (effects (font (size 1.27 1.27)) hide)
-    )
-    (pin "1")
-    (pin "2")
-    (instances
-      (project "Autko"
-        (path "/8d5cfdec-de34-4148-9100-7125640c46f5/541574ca-21e4-445f-b8e2-ded2c59d3b8a"
-          (reference "C20") (unit 1)
-        )
-      )
-    )
-  )
-  (symbol (lib_id "Device:C") (at 92.71 59.69 0) (mirror y) (unit 1)
-    (in_bom yes) (on_board yes) (dnp no)
-    (property "Reference" "C24" (at 90.17 58.42 0)
-      (effects (font (size 1.27 1.27)) (justify left))
-    )
-    (property "Value" "100nF" (at 90.17 60.96 0)
-      (effects (font (size 1.27 1.27)) (justify left))
-    )
-    (property "Footprint" "Capacitor_SMD:C_0805_2012Metric" (at 91.7448 63.5 0)
-      (effects (font (size 1.27 1.27)) hide)
-    )
-    (property "Datasheet" "~" (at 92.71 59.69 0)
-      (effects (font (size 1.27 1.27)) hide)
-    )
-    (pin "1")
-    (pin "2")
-    (instances
-      (project "Autko"
-        (path "/8d5cfdec-de34-4148-9100-7125640c46f5/541574ca-21e4-445f-b8e2-ded2c59d3b8a"
-          (reference "C24") (unit 1)
-        )
-      )
-    )
-  )
-  (symbol (lib_id "Device:C") (at 77.47 38.1 0) (unit 1)
-    (in_bom yes) (on_board yes) (dnp no)
-    (property "Reference" "C22" (at 80.01 36.83 0)
-      (effects (font (size 1.27 1.27)) (justify left))
-    )
-    (property "Value" "100nF" (at 80.01 39.37 0)
-      (effects (font (size 1.27 1.27)) (justify left))
-    )
-    (property "Footprint" "Capacitor_SMD:C_0805_2012Metric" (at 78.4352 41.91 0)
-      (effects (font (size 1.27 1.27)) hide)
-    )
-    (property "Datasheet" "~" (at 77.47 38.1 0)
-      (effects (font (size 1.27 1.27)) hide)
-    )
-    (pin "1")
-    (pin "2")
-    (instances
-      (project "Autko"
-        (path "/8d5cfdec-de34-4148-9100-7125640c46f5/541574ca-21e4-445f-b8e2-ded2c59d3b8a"
-          (reference "C22") (unit 1)
-        )
-      )
-    )
-  )
-  (symbol (lib_id "power:GND") (at 34.29 44.45 0) (unit 1)
-    (in_bom yes) (on_board yes) (dnp no)
-    (property "Reference" "#PWR041" (at 34.29 50.8 0)
-      (effects (font (size 1.27 1.27)) hide)
-    )
-    (property "Value" "GND" (at 34.29 48.26 0)
-      (effects (font (size 1.27 1.27)))
-    )
-    (property "Footprint" "" (at 34.29 44.45 0)
-      (effects (font (size 1.27 1.27)) hide)
-    )
-    (property "Datasheet" "" (at 34.29 44.45 0)
-      (effects (font (size 1.27 1.27)) hide)
-    )
-    (pin "1")
-    (instances
-      (project "Autko"
-        (path "/8d5cfdec-de34-4148-9100-7125640c46f5/541574ca-21e4-445f-b8e2-ded2c59d3b8a"
-          (reference "#PWR041") (unit 1)
-        )
-      )
-    )
-  )
   (symbol (lib_id "power:GND") (at 67.31 97.79 0) (unit 1)
     (in_bom yes) (on_board yes) (dnp no)
-    (property "Reference" "#PWR044" (at 67.31 104.14 0)
+    (property "Reference" "#PWR043" (at 67.31 104.14 0)
       (effects (font (size 1.27 1.27)) hide)
     )
@@
       (project "Autko"
         (path "/8d5cfdec-de34-4148-9100-7125640c46f5/541574ca-21e4-445f-b8e2-ded2c59d3b8a"
-          (reference "#PWR044") (unit 1)
-        )
-      )
+          (reference "#PWR043") (unit 1)
+        )
+      )

Commit message: [pcb] Remove unnecessary capacitors
Parts:
- removed C20: 10uF, Capacitor_Tantalum_SMD:CP_EIA-3216-18_Kemet-A, symbol Device:C_Polarized
Changed lines of the file:
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@@
   (junction (at 92.71 67.31) (diameter 0) (color 0 0 0 0)
   )
+  (junction (at 69.85 43.18) (diameter 0) (color 0 0 0 0)
+  )
+  (junction (at 90.17 43.18) (diameter 0) (color 0 0 0 0)
+  )
   (junction (at 46.99 33.02) (diameter 0) (color 0 0 0 0)
   )
-  (junction (at 69.85 43.18) (diameter 0) (color 0 0 0 0)
-  )
-  (junction (at 90.17 43.18) (diameter 0) (color 0 0 0 0)
-  )
-  (junction (at 34.29 43.18) (diameter 0) (color 0 0 0 0)
-  )
-  (junction (at 34.29 33.02) (diameter 0) (color 0 0 0 0)
-  )
   (wire (pts (xy 67.31 33.02) (xy 77.47 33.02))
     (stroke (width 0) (type default))
@@
     (stroke (width 0) (type default))
   )
-  (wire (pts (xy 34.29 33.02) (xy 46.99 33.02))
-    (stroke (width 0) (type default))
-  )
   (wire (pts (xy 90.17 33.02) (xy 90.17 34.29))
     (stroke (width 0) (type default))
@@
     (stroke (width 0) (type default))
   )
-  (wire (pts (xy 34.29 31.75) (xy 34.29 33.02))
-    (stroke (width 0) (type default))
-  )
   (wire (pts (xy 92.71 69.85) (xy 100.33 69.85))
     (stroke (width 0) (type default))
@@
     (stroke (width 0) (type default))
   )
-  (wire (pts (xy 34.29 43.18) (xy 34.29 44.45))
-    (stroke (width 0) (type default))
-  )
   (wire (pts (xy 81.28 64.77) (xy 81.28 67.31))
     (stroke (width 0) (type default))
@@
     (stroke (width 0) (type default))
   )
-  (wire (pts (xy 34.29 41.91) (xy 34.29 43.18))
-    (stroke (width 0) (type default))
-  )
   (wire (pts (xy 92.71 52.07) (xy 92.71 55.88))
     (stroke (width 0) (type default))
@@
     (stroke (width 0) (type default))
   )
-  (wire (pts (xy 46.99 43.18) (xy 46.99 41.91))
+  (wire (pts (xy 46.99 31.75) (xy 46.99 33.02))
+    (stroke (width 0) (type default))
+  )
+  (wire (pts (xy 46.99 41.91) (xy 46.99 44.45))
     (stroke (width 0) (type default))
   )
@@
   )
   (wire (pts (xy 81.28 67.31) (xy 92.71 67.31))
-    (stroke (width 0) (type default))
-  )
-  (wire (pts (xy 34.29 43.18) (xy 46.99 43.18))
-    (stroke (width 0) (type default))
-  )
-  (wire (pts (xy 34.29 33.02) (xy 34.29 34.29))
     (stroke (width 0) (type default))
   )
@@
     )
   )
-  (symbol (lib_id "power:+3.3V") (at 34.29 31.75 0) (unit 1)
+  (symbol (lib_id "power:+3.3V") (at 46.99 31.75 0) (unit 1)
     (in_bom yes) (on_board yes) (dnp no) (fields_autoplaced)
-    (property "Reference" "#PWR038" (at 34.29 35.56 0)
-      (effects (font (size 1.27 1.27)) hide)
-    )
-    (property "Value" "+3.3V" (at 34.29 27.94 0)
-      (effects (font (size 1.27 1.27)))
-    )
-    (property "Footprint" "" (at 34.29 31.75 0)
-      (effects (font (size 1.27 1.27)) hide)
-    )
-    (property "Datasheet" "" (at 34.29 31.75 0)
+    (property "Reference" "#PWR038" (at 46.99 35.56 0)
+      (effects (font (size 1.27 1.27)) hide)
+    )
+    (property "Value" "+3.3V" (at 46.99 27.94 0)
+      (effects (font (size 1.27 1.27)))
+    )
+    (property "Footprint" "" (at 46.99 31.75 0)
+      (effects (font (size 1.27 1.27)) hide)
+    )
+    (property "Datasheet" "" (at 46.99 31.75 0)
       (effects (font (size 1.27 1.27)) hide)
     )
@@
     )
   )
-  (symbol (lib_id "Device:C_Polarized") (at 34.29 38.1 0) (unit 1)
-    (in_bom yes) (on_board yes) (dnp no)
-    (property "Reference" "C20" (at 36.83 36.83 0)
-      (effects (font (size 1.27 1.27)) (justify left))
-    )
-    (property "Value" "10uF" (at 36.83 39.37 0)
-      (effects (font (size 1.27 1.27)) (justify left))
-    )
-    (property "Footprint" "Capacitor_Tantalum_SMD:CP_EIA-3216-18_Kemet-A" (at 35.2552 41.91 0)
-      (effects (font (size 1.27 1.27)) hide)
-    )
-    (property "Datasheet" "~" (at 34.29 38.1 0)
+  (symbol (lib_id "Device:C") (at 92.71 59.69 0) (mirror y) (unit 1)
+    (in_bom yes) (on_board yes) (dnp no)
+    (property "Reference" "C24" (at 90.17 58.42 0)
+      (effects (font (size 1.27 1.27)) (justify left))
+    )
+    (property "Value" "100nF" (at 90.17 60.96 0)
+      (effects (font (size 1.27 1.27)) (justify left))
+    )
+    (property "Footprint" "Capacitor_SMD:C_0805_2012Metric" (at 91.7448 63.5 0)
+      (effects (font (size 1.27 1.27)) hide)
+    )
+    (property "Datasheet" "~" (at 92.71 59.69 0)
       (effects (font (size 1.27 1.27)) hide)
     )
@@
       (project "Autko"
         (path "/8d5cfdec-de34-4148-9100-7125640c46f5/541574ca-21e4-445f-b8e2-ded2c59d3b8a"
-          (reference "C20") (unit 1)
-        )
-      )
-    )
-  )
-  (symbol (lib_id "Device:C") (at 92.71 59.69 0) (mirror y) (unit 1)
-    (in_bom yes) (on_board yes) (dnp no)
-    (property "Reference" "C24" (at 90.17 58.42 0)
-      (effects (font (size 1.27 1.27)) (justify left))
-    )
-    (property "Value" "100nF" (at 90.17 60.96 0)
-      (effects (font (size 1.27 1.27)) (justify left))
-    )
-    (property "Footprint" "Capacitor_SMD:C_0805_2012Metric" (at 91.7448 63.5 0)
-      (effects (font (size 1.27 1.27)) hide)
-    )
-    (property "Datasheet" "~" (at 92.71 59.69 0)
+          (reference "C24") (unit 1)
+        )
+      )
+    )
+  )
+  (symbol (lib_id "Device:C") (at 77.47 38.1 0) (unit 1)
+    (in_bom yes) (on_board yes) (dnp no)
+    (property "Reference" "C22" (at 80.01 36.83 0)
+      (effects (font (size 1.27 1.27)) (justify left))
+    )
+    (property "Value" "100nF" (at 80.01 39.37 0)
+      (effects (font (size 1.27 1.27)) (justify left))
+    )
+    (property "Footprint" "Capacitor_SMD:C_0805_2012Metric" (at 78.4352 41.91 0)
+      (effects (font (size 1.27 1.27)) hide)
+    )
+    (property "Datasheet" "~" (at 77.47 38.1 0)
       (effects (font (size 1.27 1.27)) hide)
     )
@@
       (project "Autko"
         (path "/8d5cfdec-de34-4148-9100-7125640c46f5/541574ca-21e4-445f-b8e2-ded2c59d3b8a"
-          (reference "C24") (unit 1)
-        )
-      )
-    )
-  )
-  (symbol (lib_id "Device:C") (at 77.47 38.1 0) (unit 1)
-    (in_bom yes) (on_board yes) (dnp no)
-    (property "Reference" "C22" (at 80.01 36.83 0)
-      (effects (font (size 1.27 1.27)) (justify left))
-    )
-    (property "Value" "100nF" (at 80.01 39.37 0)
-      (effects (font (size 1.27 1.27)) (justify left))
-    )
-    (property "Footprint" "Capacitor_SMD:C_0805_2012Metric" (at 78.4352 41.91 0)
-      (effects (font (size 1.27 1.27)) hide)
-    )
-    (property "Datasheet" "~" (at 77.47 38.1 0)
-      (effects (font (size 1.27 1.27)) hide)
-    )
-    (pin "1")
-    (pin "2")
-    (instances
-      (project "Autko"
-        (path "/8d5cfdec-de34-4148-9100-7125640c46f5/541574ca-21e4-445f-b8e2-ded2c59d3b8a"
           (reference "C22") (unit 1)
         )
@@
     )
   )
-  (symbol (lib_id "power:GND") (at 34.29 44.45 0) (unit 1)
-    (in_bom yes) (on_board yes) (dnp no)
-    (property "Reference" "#PWR040" (at 34.29 50.8 0)
-      (effects (font (size 1.27 1.27)) hide)
-    )
-    (property "Value" "GND" (at 34.29 48.26 0)
-      (effects (font (size 1.27 1.27)))
-    )
-    (property "Footprint" "" (at 34.29 44.45 0)
-      (effects (font (size 1.27 1.27)) hide)
-    )
-    (property "Datasheet" "" (at 34.29 44.45 0)
-      (effects (font (size 1.27 1.27)) hide)
-    )
+  (symbol (lib_id "power:GND") (at 46.99 44.45 0) (unit 1)
+    (in_bom yes) (on_board yes) (dnp no)
+    (property "Reference" "#PWR040" (at 46.99 50.8 0)
+      (effects (font (size 1.27 1.27)) hide)
+    )
+    (property "Value" "GND" (at 46.99 48.26 0)
+      (effects (font (size 1.27 1.27)))
+    )
+    (property "Footprint" "" (at 46.99 44.45 0)
+      (effects (font (size 1.27 1.27)) hide)
+    )
+    (property "Datasheet" "" (at 46.99 44.45 0)
+      (effects (font (size 1.27 1.27)) hide)
+    )

Commit message: [pcb] BT routing
Parts:
- renumbered C21 to C19, C22 to C20, C23 to C21, C24 to C22, C25 to C23
Changed lines of the file:
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@@
   (symbol (lib_id "Device:C") (at 46.99 38.1 0) (unit 1)
     (in_bom yes) (on_board yes) (dnp no)
-    (property "Reference" "C21" (at 49.53 36.83 0)
+    (property "Reference" "C19" (at 49.53 36.83 0)
       (effects (font (size 1.27 1.27)) (justify left))
     )
@@
       (project "Autko"
         (path "/8d5cfdec-de34-4148-9100-7125640c46f5/541574ca-21e4-445f-b8e2-ded2c59d3b8a"
-          (reference "C21") (unit 1)
+          (reference "C19") (unit 1)
         )
       )
@@
   (symbol (lib_id "Device:C") (at 92.71 77.47 0) (mirror y) (unit 1)
     (in_bom yes) (on_board yes) (dnp no)
-    (property "Reference" "C25" (at 90.17 76.2 0)
+    (property "Reference" "C23" (at 90.17 76.2 0)
       (effects (font (size 1.27 1.27)) (justify left))
     )
@@
       (project "Autko"
         (path "/8d5cfdec-de34-4148-9100-7125640c46f5/541574ca-21e4-445f-b8e2-ded2c59d3b8a"
-          (reference "C25") (unit 1)
+          (reference "C23") (unit 1)
         )
       )
@@
   (symbol (lib_id "Device:C") (at 92.71 59.69 0) (mirror y) (unit 1)
     (in_bom yes) (on_board yes) (dnp no)
-    (property "Reference" "C24" (at 90.17 58.42 0)
+    (property "Reference" "C22" (at 90.17 58.42 0)
       (effects (font (size 1.27 1.27)) (justify left))
     )
@@
       (project "Autko"
         (path "/8d5cfdec-de34-4148-9100-7125640c46f5/541574ca-21e4-445f-b8e2-ded2c59d3b8a"
-          (reference "C24") (unit 1)
+          (reference "C22") (unit 1)
         )
       )
@@
   (symbol (lib_id "Device:C") (at 77.47 38.1 0) (unit 1)
     (in_bom yes) (on_board yes) (dnp no)
-    (property "Reference" "C22" (at 80.01 36.83 0)
+    (property "Reference" "C20" (at 80.01 36.83 0)
       (effects (font (size 1.27 1.27)) (justify left))
     )
@@
       (project "Autko"
         (path "/8d5cfdec-de34-4148-9100-7125640c46f5/541574ca-21e4-445f-b8e2-ded2c59d3b8a"
-          (reference "C22") (unit 1)
+          (reference "C20") (unit 1)
         )
       )
@@
   (symbol (lib_id "Device:C_Polarized") (at 90.17 38.1 0) (unit 1)
     (in_bom yes) (on_board yes) (dnp no)
-    (property "Reference" "C23" (at 92.71 36.83 0)
+    (property "Reference" "C21" (at 92.71 36.83 0)
       (effects (font (size 1.27 1.27)) (justify left))
     )
@@
       (project "Autko"
         (path "/8d5cfdec-de34-4148-9100-7125640c46f5/541574ca-21e4-445f-b8e2-ded2c59d3b8a"
-          (reference "C23") (unit 1)
-        )
-      )
+          (reference "C21") (unit 1)
+        )
+      )

Commit message: [pcb] Some power routing
Connections:
- net at C23.1, U11.11 (BO1), U11.12 (BO1): now also M2.2 (+); no longer M2.1 (+)
- net at C23.2, U11.7 (BO2), U11.8 (BO2): now also M2.1 (-); no longer M2.2 (-)
Changed lines of the file:
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@@
     (effects (font (size 1.27 1.27)) (justify right))
   )
-  (symbol (lib_id "Motor:Motor_DC") (at 100.33 76.2 0) (unit 1)
+  (symbol (lib_name "Motor_DC_1") (lib_id "Motor:Motor_DC") (at 100.33 76.2 0) (unit 1)
     (in_bom yes) (on_board yes) (dnp no) (fields_autoplaced)
     (property "Reference" "M2" (at 105.41 78.105 0)
