File: pcb/Line_sensors.kicad_sch (KiCad schematic)
At the start: 31 parts, among them Q2 BC817, U10 CNY70, U11 CNY70, U5 CNY70, U6 CNY70, U7 CNY70, U8 CNY70, U9 CNY70

Commit message: Power switch footprint and initial pcb
Parts:
- renumbered U11 to U10, U5 to U4, U6 to U5, U7 to U6, U8 to U7, U9 to U8, U10 to U9
Changed lines of the file:
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@@
   (symbol (lib_id "power:GND") (at 93.98 49.53 0) (unit 1)
     (in_bom yes) (on_board yes) (dnp no)
-    (property "Reference" "#PWR032" (at 93.98 55.88 0)
+    (property "Reference" "#PWR031" (at 93.98 55.88 0)
       (effects (font (size 1.27 1.27)) hide)
     )
@@
       (project "Autko"
         (path "/8d5cfdec-de34-4148-9100-7125640c46f5/80d635c6-4a73-4538-989a-c930c6a7f33b"
-          (reference "#PWR032") (unit 1)
+          (reference "#PWR031") (unit 1)
         )
       )
@@
   (symbol (lib_id "power:GND") (at 59.69 49.53 0) (unit 1)
     (in_bom yes) (on_board yes) (dnp no)
-    (property "Reference" "#PWR031" (at 59.69 55.88 0)
+    (property "Reference" "#PWR030" (at 59.69 55.88 0)
       (effects (font (size 1.27 1.27)) hide)
     )
@@
       (project "Autko"
         (path "/8d5cfdec-de34-4148-9100-7125640c46f5/80d635c6-4a73-4538-989a-c930c6a7f33b"
-          (reference "#PWR031") (unit 1)
+          (reference "#PWR030") (unit 1)
         )
       )
@@
   (symbol (lib_id "power:+3.3V") (at 41.91 26.67 0) (unit 1)
     (in_bom yes) (on_board yes) (dnp no) (fields_autoplaced)
-    (property "Reference" "#PWR030" (at 41.91 30.48 0)
+    (property "Reference" "#PWR029" (at 41.91 30.48 0)
       (effects (font (size 1.27 1.27)) hide)
     )
@@
       (project "Autko"
         (path "/8d5cfdec-de34-4148-9100-7125640c46f5/80d635c6-4a73-4538-989a-c930c6a7f33b"
-          (reference "#PWR030") (unit 1)
+          (reference "#PWR029") (unit 1)
         )
       )
@@
   (symbol (lib_id "Sensor_Proximity:CNY70") (at 85.09 45.72 0) (unit 1)
     (in_bom yes) (on_board yes) (dnp no) (fields_autoplaced)
-    (property "Reference" "U6" (at 85.09 38.1 0)
+    (property "Reference" "U5" (at 85.09 38.1 0)
       (effects (font (size 1.27 1.27)))
     )
@@
       (project "Autko"
         (path "/8d5cfdec-de34-4148-9100-7125640c46f5/80d635c6-4a73-4538-989a-c930c6a7f33b"
-          (reference "U6") (unit 1)
+          (reference "U5") (unit 1)
         )
       )
@@
   (symbol (lib_id "power:GND") (at 128.27 49.53 0) (unit 1)
     (in_bom yes) (on_board yes) (dnp no)
-    (property "Reference" "#PWR033" (at 128.27 55.88 0)
+    (property "Reference" "#PWR032" (at 128.27 55.88 0)
       (effects (font (size 1.27 1.27)) hide)
     )
@@
       (project "Autko"
         (path "/8d5cfdec-de34-4148-9100-7125640c46f5/80d635c6-4a73-4538-989a-c930c6a7f33b"
-          (reference "#PWR033") (unit 1)
+          (reference "#PWR032") (unit 1)
         )
       )
@@
   (symbol (lib_id "Sensor_Proximity:CNY70") (at 119.38 45.72 0) (unit 1)
     (in_bom yes) (on_board yes) (dnp no) (fields_autoplaced)
-    (property "Reference" "U7" (at 119.38 38.1 0)
+    (property "Reference" "U6" (at 119.38 38.1 0)
       (effects (font (size 1.27 1.27)))
     )
@@
       (project "Autko"
         (path "/8d5cfdec-de34-4148-9100-7125640c46f5/80d635c6-4a73-4538-989a-c930c6a7f33b"
-          (reference "U7") (unit 1)
+          (reference "U6") (unit 1)
         )
       )
@@
   (symbol (lib_id "power:GND") (at 196.85 49.53 0) (unit 1)
     (in_bom yes) (on_board yes) (dnp no)
-    (property "Reference" "#PWR035" (at 196.85 55.88 0)
+    (property "Reference" "#PWR034" (at 196.85 55.88 0)
       (effects (font (size 1.27 1.27)) hide)
     )
@@
       (project "Autko"
         (path "/8d5cfdec-de34-4148-9100-7125640c46f5/80d635c6-4a73-4538-989a-c930c6a7f33b"
-          (reference "#PWR035") (unit 1)
+          (reference "#PWR034") (unit 1)
         )
       )
@@
   (symbol (lib_id "Sensor_Proximity:CNY70") (at 153.67 45.72 0) (unit 1)
     (in_bom yes) (on_board yes) (dnp no) (fields_autoplaced)
-    (property "Reference" "U8" (at 153.67 38.1 0)
+    (property "Reference" "U7" (at 153.67 38.1 0)
       (effects (font (size 1.27 1.27)))
     )
@@
       (project "Autko"
         (path "/8d5cfdec-de34-4148-9100-7125640c46f5/80d635c6-4a73-4538-989a-c930c6a7f33b"
-          (reference "U8") (unit 1)
+          (reference "U7") (unit 1)
         )
       )
@@
   (symbol (lib_id "power:GND") (at 162.56 49.53 0) (unit 1)
     (in_bom yes) (on_board yes) (dnp no)
-    (property "Reference" "#PWR034" (at 162.56 55.88 0)
+    (property "Reference" "#PWR033" (at 162.56 55.88 0)
       (effects (font (size 1.27 1.27)) hide)
     )
@@
       (project "Autko"
         (path "/8d5cfdec-de34-4148-9100-7125640c46f5/80d635c6-4a73-4538-989a-c930c6a7f33b"
-          (reference "#PWR034") (unit 1)
+          (reference "#PWR033") (unit 1)
         )
       )
@@
   (symbol (lib_id "Sensor_Proximity:CNY70") (at 50.8 45.72 0) (unit 1)
     (in_bom yes) (on_board yes) (dnp no) (fields_autoplaced)
-    (property "Reference" "U5" (at 50.8 38.1 0)
+    (property "Reference" "U4" (at 50.8 38.1 0)
       (effects (font (size 1.27 1.27)))
     )
@@
       (project "Autko"
         (path "/8d5cfdec-de34-4148-9100-7125640c46f5/80d635c6-4a73-4538-989a-c930c6a7f33b"
-          (reference "U5") (unit 1)
+          (reference "U4") (unit 1)
         )
       )
@@
   (symbol (lib_id "Sensor_Proximity:CNY70") (at 222.25 45.72 0) (unit 1)
     (in_bom yes) (on_board yes) (dnp no) (fields_autoplaced)
-    (property "Reference" "U10" (at 222.25 38.1 0)
+    (property "Reference" "U9" (at 222.25 38.1 0)
       (effects (font (size 1.27 1.27)))
     )
@@
       (project "Autko"
         (path "/8d5cfdec-de34-4148-9100-7125640c46f5/80d635c6-4a73-4538-989a-c930c6a7f33b"
-          (reference "U10") (unit 1)
+          (reference "U9") (unit 1)
         )
       )
@@
   (symbol (lib_id "power:GND") (at 41.91 69.85 0) (unit 1)
     (in_bom yes) (on_board yes) (dnp no)
-    (property "Reference" "#PWR038" (at 41.91 76.2 0)
+    (property "Reference" "#PWR037" (at 41.91 76.2 0)
       (effects (font (size 1.27 1.27)) hide)
     )
@@
       (project "Autko"
         (path "/8d5cfdec-de34-4148-9100-7125640c46f5/80d635c6-4a73-4538-989a-c930c6a7f33b"
-          (reference "#PWR038") (unit 1)
+          (reference "#PWR037") (unit 1)
         )
       )
@@
   (symbol (lib_id "power:GND") (at 231.14 49.53 0) (unit 1)
     (in_bom yes) (on_board yes) (dnp no)
-    (property "Reference" "#PWR036" (at 231.14 55.88 0)
+    (property "Reference" "#PWR035" (at 231.14 55.88 0)
       (effects (font (size 1.27 1.27)) hide)
     )
@@
       (project "Autko"
         (path "/8d5cfdec-de34-4148-9100-7125640c46f5/80d635c6-4a73-4538-989a-c930c6a7f33b"
+          (reference "#PWR035") (unit 1)
+        )
+      )
+    )
+  )
+  (symbol (lib_id "power:GND") (at 265.43 49.53 0) (unit 1)
+    (in_bom yes) (on_board yes) (dnp no)
+    (property "Reference" "#PWR036" (at 265.43 55.88 0)
+      (effects (font (size 1.27 1.27)) hide)
+    )
+    (property "Value" "GND" (at 265.43 53.34 0)
+      (effects (font (size 1.27 1.27)))
+    )
+    (property "Footprint" "" (at 265.43 49.53 0)
+      (effects (font (size 1.27 1.27)) hide)
+    )
+    (property "Datasheet" "" (at 265.43 49.53 0)
+      (effects (font (size 1.27 1.27)) hide)
+    )
+    (pin "1")
+    (instances
+      (project "Autko"
+        (path "/8d5cfdec-de34-4148-9100-7125640c46f5/80d635c6-4a73-4538-989a-c930c6a7f33b"
           (reference "#PWR036") (unit 1)
-        )
-      )
-    )
-  )
-  (symbol (lib_id "power:GND") (at 265.43 49.53 0) (unit 1)
-    (in_bom yes) (on_board yes) (dnp no)
-    (property "Reference" "#PWR037" (at 265.43 55.88 0)
-      (effects (font (size 1.27 1.27)) hide)
-    )
-    (property "Value" "GND" (at 265.43 53.34 0)
-      (effects (font (size 1.27 1.27)))
-    )
-    (property "Footprint" "" (at 265.43 49.53 0)
-      (effects (font (size 1.27 1.27)) hide)
-    )
-    (property "Datasheet" "" (at 265.43 49.53 0)
-      (effects (font (size 1.27 1.27)) hide)
-    )
-    (pin "1")
-    (instances
-      (project "Autko"
-        (path "/8d5cfdec-de34-4148-9100-7125640c46f5/80d635c6-4a73-4538-989a-c930c6a7f33b"
-          (reference "#PWR037") (unit 1)
         )
       )
@@
   (symbol (lib_id "Sensor_Proximity:CNY70") (at 256.54 45.72 0) (unit 1)
     (in_bom yes) (on_board yes) (dnp no) (fields_autoplaced)
-    (property "Reference" "U11" (at 256.54 38.1 0)
+    (property "Reference" "U10" (at 256.54 38.1 0)
       (effects (font (size 1.27 1.27)))
     )
@@
       (project "Autko"
         (path "/8d5cfdec-de34-4148-9100-7125640c46f5/80d635c6-4a73-4538-989a-c930c6a7f33b"
-          (reference "U11") (unit 1)
+          (reference "U10") (unit 1)
         )
       )
@@
   (symbol (lib_id "Sensor_Proximity:CNY70") (at 187.96 45.72 0) (unit 1)
     (in_bom yes) (on_board yes) (dnp no) (fields_autoplaced)
-    (property "Reference" "U9" (at 187.96 38.1 0)
+    (property "Reference" "U8" (at 187.96 38.1 0)
       (effects (font (size 1.27 1.27)))
     )
@@
       (project "Autko"
         (path "/8d5cfdec-de34-4148-9100-7125640c46f5/80d635c6-4a73-4538-989a-c930c6a7f33b"
-          (reference "U9") (unit 1)
-        )
-      )
+          (reference "U8") (unit 1)
+        )
+      )

Commit message: [pcb] BT routing
Parts:
- renumbered R23 to R22, R24 to R23, R25 to R24, R26 to R25, R27 to R26, R28 to R27, R29 to R28, R30 to R29, R31 to R30, R32 to R31, R33 to R32, R34 to R33, R35 to R34, R36 to R35, R37 to R36
Changed lines of the file:
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@@
   (symbol (lib_id "Device:R") (at 33.02 58.42 0) (mirror y) (unit 1)
     (in_bom yes) (on_board yes) (dnp no)
-    (property "Reference" "R37" (at 30.48 57.15 0)
+    (property "Reference" "R36" (at 30.48 57.15 0)
       (effects (font (size 1.27 1.27)) (justify left))
     )
@@
       (project "Autko"
         (path "/8d5cfdec-de34-4148-9100-7125640c46f5/80d635c6-4a73-4538-989a-c930c6a7f33b"
-          (reference "R37") (unit 1)
+          (reference "R36") (unit 1)
         )
       )
@@
   (symbol (lib_id "Device:R") (at 247.65 33.02 0) (unit 1)
     (in_bom yes) (on_board yes) (dnp no)
-    (property "Reference" "R35" (at 250.19 31.75 0)
+    (property "Reference" "R34" (at 250.19 31.75 0)
       (effects (font (size 1.27 1.27)) (justify left))
     )
@@
       (project "Autko"
         (path "/8d5cfdec-de34-4148-9100-7125640c46f5/80d635c6-4a73-4538-989a-c930c6a7f33b"
-          (reference "R35") (unit 1)
+          (reference "R34") (unit 1)
         )
       )
@@
   (symbol (lib_id "Device:R") (at 144.78 33.02 0) (unit 1)
     (in_bom yes) (on_board yes) (dnp no)
-    (property "Reference" "R29" (at 147.32 31.75 0)
+    (property "Reference" "R28" (at 147.32 31.75 0)
       (effects (font (size 1.27 1.27)) (justify left))
     )
@@
       (project "Autko"
         (path "/8d5cfdec-de34-4148-9100-7125640c46f5/80d635c6-4a73-4538-989a-c930c6a7f33b"
-          (reference "R29") (unit 1)
+          (reference "R28") (unit 1)
         )
       )
@@
   (symbol (lib_id "Device:R") (at 41.91 33.02 0) (unit 1)
     (in_bom yes) (on_board yes) (dnp no)
-    (property "Reference" "R23" (at 44.45 31.75 0)
+    (property "Reference" "R22" (at 44.45 31.75 0)
       (effects (font (size 1.27 1.27)) (justify left))
     )
@@
       (project "Autko"
         (path "/8d5cfdec-de34-4148-9100-7125640c46f5/80d635c6-4a73-4538-989a-c930c6a7f33b"
-          (reference "R23") (unit 1)
+          (reference "R22") (unit 1)
         )
       )
@@
   (symbol (lib_id "Device:R") (at 63.5 33.02 0) (unit 1)
     (in_bom yes) (on_board yes) (dnp no)
-    (property "Reference" "R24" (at 66.04 31.75 0)
+    (property "Reference" "R23" (at 66.04 31.75 0)
       (effects (font (size 1.27 1.27)) (justify left))
     )
@@
       (project "Autko"
         (path "/8d5cfdec-de34-4148-9100-7125640c46f5/80d635c6-4a73-4538-989a-c930c6a7f33b"
+          (reference "R23") (unit 1)
+        )
+      )
+    )
+  )
+  (symbol (lib_id "Device:R") (at 76.2 33.02 0) (unit 1)
+    (in_bom yes) (on_board yes) (dnp no)
+    (property "Reference" "R24" (at 78.74 31.75 0)
+      (effects (font (size 1.27 1.27)) (justify left))
+    )
+    (property "Value" "220R" (at 78.74 34.29 0)
+      (effects (font (size 1.27 1.27)) (justify left))
+    )
+    (property "Footprint" "Resistor_SMD:R_0805_2012Metric" (at 74.422 33.02 90)
+      (effects (font (size 1.27 1.27)) hide)
+    )
+    (property "Datasheet" "~" (at 76.2 33.02 0)
+      (effects (font (size 1.27 1.27)) hide)
+    )
+    (pin "1")
+    (pin "2")
+    (instances
+      (project "Autko"
+        (path "/8d5cfdec-de34-4148-9100-7125640c46f5/80d635c6-4a73-4538-989a-c930c6a7f33b"
           (reference "R24") (unit 1)
         )
@@
     )
   )
-  (symbol (lib_id "Device:R") (at 76.2 33.02 0) (unit 1)
-    (in_bom yes) (on_board yes) (dnp no)
-    (property "Reference" "R25" (at 78.74 31.75 0)
-      (effects (font (size 1.27 1.27)) (justify left))
-    )
-    (property "Value" "220R" (at 78.74 34.29 0)
-      (effects (font (size 1.27 1.27)) (justify left))
-    )
-    (property "Footprint" "Resistor_SMD:R_0805_2012Metric" (at 74.422 33.02 90)
-      (effects (font (size 1.27 1.27)) hide)
-    )
-    (property "Datasheet" "~" (at 76.2 33.02 0)
-      (effects (font (size 1.27 1.27)) hide)
-    )
-    (pin "1")
-    (pin "2")
-    (instances
-      (project "Autko"
-        (path "/8d5cfdec-de34-4148-9100-7125640c46f5/80d635c6-4a73-4538-989a-c930c6a7f33b"
-          (reference "R25") (unit 1)
-        )
-      )
-    )
-  )
   (symbol (lib_id "Device:R") (at 110.49 33.02 0) (unit 1)
     (in_bom yes) (on_board yes) (dnp no)
-    (property "Reference" "R27" (at 113.03 31.75 0)
+    (property "Reference" "R26" (at 113.03 31.75 0)
       (effects (font (size 1.27 1.27)) (justify left))
     )
@@
       (project "Autko"
         (path "/8d5cfdec-de34-4148-9100-7125640c46f5/80d635c6-4a73-4538-989a-c930c6a7f33b"
-          (reference "R27") (unit 1)
+          (reference "R26") (unit 1)
         )
       )
@@
   (symbol (lib_id "Device:R") (at 166.37 33.02 0) (unit 1)
     (in_bom yes) (on_board yes) (dnp no)
-    (property "Reference" "R30" (at 168.91 31.75 0)
+    (property "Reference" "R29" (at 168.91 31.75 0)
       (effects (font (size 1.27 1.27)) (justify left))
     )
@@
       (project "Autko"
         (path "/8d5cfdec-de34-4148-9100-7125640c46f5/80d635c6-4a73-4538-989a-c930c6a7f33b"
-          (reference "R30") (unit 1)
+          (reference "R29") (unit 1)
         )
       )
@@
   (symbol (lib_id "Device:R") (at 234.95 33.02 0) (unit 1)
     (in_bom yes) (on_board yes) (dnp no)
-    (property "Reference" "R34" (at 237.49 31.75 0)
+    (property "Reference" "R33" (at 237.49 31.75 0)
       (effects (font (size 1.27 1.27)) (justify left))
     )
@@
       (project "Autko"
         (path "/8d5cfdec-de34-4148-9100-7125640c46f5/80d635c6-4a73-4538-989a-c930c6a7f33b"
-          (reference "R34") (unit 1)
+          (reference "R33") (unit 1)
         )
       )
@@
   (symbol (lib_id "Device:R") (at 179.07 33.02 0) (unit 1)
     (in_bom yes) (on_board yes) (dnp no)
-    (property "Reference" "R31" (at 181.61 31.75 0)
+    (property "Reference" "R30" (at 181.61 31.75 0)
       (effects (font (size 1.27 1.27)) (justify left))
     )
@@
       (project "Autko"
         (path "/8d5cfdec-de34-4148-9100-7125640c46f5/80d635c6-4a73-4538-989a-c930c6a7f33b"
-          (reference "R31") (unit 1)
+          (reference "R30") (unit 1)
         )
       )
@@
   (symbol (lib_id "Device:R") (at 97.79 33.02 0) (unit 1)
     (in_bom yes) (on_board yes) (dnp no)
-    (property "Reference" "R26" (at 100.33 31.75 0)
+    (property "Reference" "R25" (at 100.33 31.75 0)
       (effects (font (size 1.27 1.27)) (justify left))
     )
@@
       (project "Autko"
         (path "/8d5cfdec-de34-4148-9100-7125640c46f5/80d635c6-4a73-4538-989a-c930c6a7f33b"
-          (reference "R26") (unit 1)
+          (reference "R25") (unit 1)
         )
       )
@@
   (symbol (lib_id "Device:R") (at 200.66 33.02 0) (unit 1)
     (in_bom yes) (on_board yes) (dnp no)
-    (property "Reference" "R32" (at 203.2 31.75 0)
+    (property "Reference" "R31" (at 203.2 31.75 0)
       (effects (font (size 1.27 1.27)) (justify left))
     )
@@
       (project "Autko"
         (path "/8d5cfdec-de34-4148-9100-7125640c46f5/80d635c6-4a73-4538-989a-c930c6a7f33b"
+          (reference "R31") (unit 1)
+        )
+      )
+    )
+  )
+  (symbol (lib_id "Device:R") (at 213.36 33.02 0) (unit 1)
+    (in_bom yes) (on_board yes) (dnp no)
+    (property "Reference" "R32" (at 215.9 31.75 0)
+      (effects (font (size 1.27 1.27)) (justify left))
+    )
+    (property "Value" "220R" (at 215.9 34.29 0)
+      (effects (font (size 1.27 1.27)) (justify left))
+    )
+    (property "Footprint" "Resistor_SMD:R_0805_2012Metric" (at 211.582 33.02 90)
+      (effects (font (size 1.27 1.27)) hide)
+    )
+    (property "Datasheet" "~" (at 213.36 33.02 0)
+      (effects (font (size 1.27 1.27)) hide)
+    )
+    (pin "1")
+    (pin "2")
+    (instances
+      (project "Autko"
+        (path "/8d5cfdec-de34-4148-9100-7125640c46f5/80d635c6-4a73-4538-989a-c930c6a7f33b"
           (reference "R32") (unit 1)
-        )
-      )
-    )
-  )
-  (symbol (lib_id "Device:R") (at 213.36 33.02 0) (unit 1)
-    (in_bom yes) (on_board yes) (dnp no)
-    (property "Reference" "R33" (at 215.9 31.75 0)
-      (effects (font (size 1.27 1.27)) (justify left))
-    )
-    (property "Value" "220R" (at 215.9 34.29 0)
-      (effects (font (size 1.27 1.27)) (justify left))
-    )
-    (property "Footprint" "Resistor_SMD:R_0805_2012Metric" (at 211.582 33.02 90)
-      (effects (font (size 1.27 1.27)) hide)
-    )
-    (property "Datasheet" "~" (at 213.36 33.02 0)
-      (effects (font (size 1.27 1.27)) hide)
-    )
-    (pin "1")
-    (pin "2")
-    (instances
-      (project "Autko"
-        (path "/8d5cfdec-de34-4148-9100-7125640c46f5/80d635c6-4a73-4538-989a-c930c6a7f33b"
-          (reference "R33") (unit 1)
         )
       )
@@
   (symbol (lib_id "Device:R") (at 269.24 33.02 0) (unit 1)
     (in_bom yes) (on_board yes) (dnp no)
-    (property "Reference" "R36" (at 271.78 31.75 0)
+    (property "Reference" "R35" (at 271.78 31.75 0)
       (effects (font (size 1.27 1.27)) (justify left))
     )
@@
       (project "Autko"
         (path "/8d5cfdec-de34-4148-9100-7125640c46f5/80d635c6-4a73-4538-989a-c930c6a7f33b"
-          (reference "R36") (unit 1)
+          (reference "R35") (unit 1)
         )
       )
@@
   (symbol (lib_id "Device:R") (at 132.08 33.02 0) (unit 1)
     (in_bom yes) (on_board yes) (dnp no)
-    (property "Reference" "R28" (at 134.62 31.75 0)
+    (property "Reference" "R27" (at 134.62 31.75 0)
       (effects (font (size 1.27 1.27)) (justify left))
     )
@@
       (project "Autko"
         (path "/8d5cfdec-de34-4148-9100-7125640c46f5/80d635c6-4a73-4538-989a-c930c6a7f33b"
-          (reference "R28") (unit 1)
-        )
-      )
+          (reference "R27") (unit 1)
+        )
+      )

Commit message: [pcb] Line sensors routed
Parts:
- U10, U4, U5, U6, U7, U8, U9: footprint OptoDevice:Vishay_CNY70 -> Autko:Vishay_CNY70
Changed lines of the file:
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@@
       (effects (font (size 1.27 1.27)))
     )
-    (property "Footprint" "OptoDevice:Vishay_CNY70" (at 85.09 50.8 0)
+    (property "Footprint" "Autko:Vishay_CNY70" (at 85.09 50.8 0)
       (effects (font (size 1.27 1.27)) hide)
     )
@@
       (effects (font (size 1.27 1.27)))
     )
-    (property "Footprint" "OptoDevice:Vishay_CNY70" (at 119.38 50.8 0)
+    (property "Footprint" "Autko:Vishay_CNY70" (at 119.38 50.8 0)
       (effects (font (size 1.27 1.27)) hide)
     )
@@
       (effects (font (size 1.27 1.27)))
     )
-    (property "Footprint" "OptoDevice:Vishay_CNY70" (at 153.67 50.8 0)
+    (property "Footprint" "Autko:Vishay_CNY70" (at 153.67 50.8 0)
       (effects (font (size 1.27 1.27)) hide)
     )
@@
       (effects (font (size 1.27 1.27)))
     )
-    (property "Footprint" "OptoDevice:Vishay_CNY70" (at 50.8 50.8 0)
+    (property "Footprint" "Autko:Vishay_CNY70" (at 50.8 50.8 0)
       (effects (font (size 1.27 1.27)) hide)
     )
@@
       (effects (font (size 1.27 1.27)))
     )
-    (property "Footprint" "OptoDevice:Vishay_CNY70" (at 222.25 50.8 0)
+    (property "Footprint" "Autko:Vishay_CNY70" (at 222.25 50.8 0)
       (effects (font (size 1.27 1.27)) hide)
     )
@@
       (effects (font (size 1.27 1.27)))
     )
-    (property "Footprint" "OptoDevice:Vishay_CNY70" (at 256.54 50.8 0)
+    (property "Footprint" "Autko:Vishay_CNY70" (at 256.54 50.8 0)
       (effects (font (size 1.27 1.27)) hide)
     )
@@
       (effects (font (size 1.27 1.27)))
     )
-    (property "Footprint" "OptoDevice:Vishay_CNY70" (at 187.96 50.8 0)
-      (effects (font (size 1.27 1.27)) hide)
-    )
+    (property "Footprint" "Autko:Vishay_CNY70" (at 187.96 50.8 0)
+      (effects (font (size 1.27 1.27)) hide)
+    )
