File: pcb/Microcontroller.kicad_sch (KiCad schematic)
At the start: 36 parts, among them J1 PDI, SW2 START, SW3 STOP, U3 ATxmega16A4U-A, X1 8MHz

Commit message: [pcb] Voltage regulator changed to TLV761
Parts:
- C15: footprint Capacitor_Tantalum_SMD:CP_EIA-3528-12_Kemet-T -> Capacitor_Tantalum_SMD:CP_EIA-3216-18_Kemet-A
Changed lines of the file:
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@@
       (effects (font (size 1.27 1.27)) (justify left))
     )
-    (property "Footprint" "Capacitor_Tantalum_SMD:CP_EIA-3528-12_Kemet-T" (at 89.8652 36.83 0)
+    (property "Footprint" "Capacitor_Tantalum_SMD:CP_EIA-3216-18_Kemet-A" (at 89.8652 36.83 0)
       (effects (font (size 1.27 1.27)) hide)
     )

Commit message: [pcb] Assign smaller footprints
Parts:
- C10, C11, C12, C13, C14, C16, C17, C18: footprint Capacitor_SMD:C_0805_2012Metric -> Capacitor_SMD:C_0603_1608Metric
- C15: footprint Capacitor_Tantalum_SMD:CP_EIA-3216-18_Kemet-A -> Capacitor_SMD:C_1206_3216Metric
- D10, D11, D5, D6, D7, D8, D9: footprint LED_SMD:LED_0805_2012Metric -> LED_SMD:LED_0603_1608Metric
- FB1: footprint Capacitor_SMD:C_0805_2012Metric -> Inductor_SMD:L_0603_1608Metric
- R10, R11, R12, R13, R14, R15, R16, R17, R18, R19, R20, R21, R8, R9: footprint Resistor_SMD:R_0805_2012Metric -> Resistor_SMD:R_0603_1608Metric
Changed lines of the file:
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@@
       (effects (font (size 1.27 1.27)) (justify left))
     )
-    (property "Footprint" "Resistor_SMD:R_0805_2012Metric" (at 137.922 90.17 90)
+    (property "Footprint" "Resistor_SMD:R_0603_1608Metric" (at 137.922 90.17 90)
       (effects (font (size 1.27 1.27)) hide)
     )
@@
       (effects (font (size 1.27 1.27)) (justify right))
     )
-    (property "Footprint" "LED_SMD:LED_0805_2012Metric" (at 165.1 81.28 0)
+    (property "Footprint" "LED_SMD:LED_0603_1608Metric" (at 165.1 81.28 0)
       (effects (font (size 1.27 1.27)) hide)
     )
@@
       (effects (font (size 1.27 1.27)) (justify right))
     )
-    (property "Footprint" "LED_SMD:LED_0805_2012Metric" (at 177.8 81.28 0)
+    (property "Footprint" "LED_SMD:LED_0603_1608Metric" (at 177.8 81.28 0)
       (effects (font (size 1.27 1.27)) hide)
     )
@@
       (effects (font (size 1.27 1.27)) (justify right))
     )
-    (property "Footprint" "LED_SMD:LED_0805_2012Metric" (at 203.2 81.28 0)
+    (property "Footprint" "LED_SMD:LED_0603_1608Metric" (at 203.2 81.28 0)
       (effects (font (size 1.27 1.27)) hide)
     )
@@
       (effects (font (size 1.27 1.27)))
     )
-    (property "Footprint" "Resistor_SMD:R_0805_2012Metric" (at 212.09 41.148 90)
+    (property "Footprint" "Resistor_SMD:R_0603_1608Metric" (at 212.09 41.148 90)
       (effects (font (size 1.27 1.27)) hide)
     )
@@
       (effects (font (size 1.27 1.27)) (justify left))
     )
-    (property "Footprint" "Capacitor_SMD:C_0805_2012Metric" (at 59.3852 36.83 0)
+    (property "Footprint" "Capacitor_SMD:C_0603_1608Metric" (at 59.3852 36.83 0)
       (effects (font (size 1.27 1.27)) hide)
     )
@@
       (effects (font (size 1.27 1.27)) (justify left))
     )
-    (property "Footprint" "Capacitor_SMD:C_0805_2012Metric" (at 77.1652 36.83 0)
+    (property "Footprint" "Capacitor_SMD:C_0603_1608Metric" (at 77.1652 36.83 0)
       (effects (font (size 1.27 1.27)) hide)
     )
@@
       (effects (font (size 1.27 1.27)))
     )
-    (property "Footprint" "Capacitor_SMD:C_0805_2012Metric" (at 82.55 29.718 90)
+    (property "Footprint" "Inductor_SMD:L_0603_1608Metric" (at 82.55 29.718 90)
       (effects (font (size 1.27 1.27)) hide)
     )
@@
       (effects (font (size 1.27 1.27)) (justify left))
     )
-    (property "Footprint" "Resistor_SMD:R_0805_2012Metric" (at 216.662 44.45 90)
+    (property "Footprint" "Resistor_SMD:R_0603_1608Metric" (at 216.662 44.45 90)
       (effects (font (size 1.27 1.27)) hide)
     )
@@
       (effects (font (size 1.27 1.27)))
     )
-    (property "Footprint" "Resistor_SMD:R_0805_2012Metric" (at 30.48 50.038 90)
+    (property "Footprint" "Resistor_SMD:R_0603_1608Metric" (at 30.48 50.038 90)
       (effects (font (size 1.27 1.27)) hide)
     )
@@
       (effects (font (size 1.27 1.27)) (justify right))
     )
-    (property "Footprint" "LED_SMD:LED_0805_2012Metric" (at 139.7 81.28 0)
+    (property "Footprint" "LED_SMD:LED_0603_1608Metric" (at 139.7 81.28 0)
       (effects (font (size 1.27 1.27)) hide)
     )
@@
       (effects (font (size 1.27 1.27)) (justify left))
     )
-    (property "Footprint" "Resistor_SMD:R_0805_2012Metric" (at 183.642 44.45 90)
+    (property "Footprint" "Resistor_SMD:R_0603_1608Metric" (at 183.642 44.45 90)
       (effects (font (size 1.27 1.27)) hide)
     )
@@
       (effects (font (size 1.27 1.27)) (justify left))
     )
-    (property "Footprint" "Capacitor_SMD:C_0805_2012Metric" (at 206.7052 48.26 0)
+    (property "Footprint" "Capacitor_SMD:C_0603_1608Metric" (at 206.7052 48.26 0)
       (effects (font (size 1.27 1.27)) hide)
     )
@@
       (effects (font (size 1.27 1.27)) (justify right))
     )
-    (property "Footprint" "LED_SMD:LED_0805_2012Metric" (at 190.5 81.28 0)
+    (property "Footprint" "LED_SMD:LED_0603_1608Metric" (at 190.5 81.28 0)
       (effects (font (size 1.27 1.27)) hide)
     )
@@
       (effects (font (size 1.27 1.27)) (justify left))
     )
-    (property "Footprint" "Capacitor_SMD:C_0805_2012Metric" (at 47.9552 36.83 0)
+    (property "Footprint" "Capacitor_SMD:C_0603_1608Metric" (at 47.9552 36.83 0)
       (effects (font (size 1.27 1.27)) hide)
     )
@@
       (effects (font (size 1.27 1.27)) (justify left))
     )
-    (property "Footprint" "Resistor_SMD:R_0805_2012Metric" (at 176.022 90.17 90)
+    (property "Footprint" "Resistor_SMD:R_0603_1608Metric" (at 176.022 90.17 90)
       (effects (font (size 1.27 1.27)) hide)
     )
@@
       (effects (font (size 1.27 1.27)) (justify left))
     )
-    (property "Footprint" "Resistor_SMD:R_0805_2012Metric" (at 214.122 90.17 90)
+    (property "Footprint" "Resistor_SMD:R_0603_1608Metric" (at 214.122 90.17 90)
       (effects (font (size 1.27 1.27)) hide)
     )
@@
       (effects (font (size 1.27 1.27)))
     )
-    (property "Footprint" "Resistor_SMD:R_0805_2012Metric" (at 179.07 41.148 90)
+    (property "Footprint" "Resistor_SMD:R_0603_1608Metric" (at 179.07 41.148 90)
       (effects (font (size 1.27 1.27)) hide)
     )
@@
       (effects (font (size 1.27 1.27)) (justify left))
     )
-    (property "Footprint" "Resistor_SMD:R_0805_2012Metric" (at 163.322 90.17 90)
+    (property "Footprint" "Resistor_SMD:R_0603_1608Metric" (at 163.322 90.17 90)
       (effects (font (size 1.27 1.27)) hide)
     )
@@
       (effects (font (size 1.27 1.27)) (justify left))
     )
-    (property "Footprint" "Capacitor_SMD:C_0805_2012Metric" (at 173.6852 48.26 0)
+    (property "Footprint" "Capacitor_SMD:C_0603_1608Metric" (at 173.6852 48.26 0)
       (effects (font (size 1.27 1.27)) hide)
     )
@@
       (effects (font (size 1.27 1.27)) (justify left))
     )
-    (property "Footprint" "Resistor_SMD:R_0805_2012Metric" (at 103.632 74.93 90)
+    (property "Footprint" "Resistor_SMD:R_0603_1608Metric" (at 103.632 74.93 90)
       (effects (font (size 1.27 1.27)) hide)
     )
@@
       (effects (font (size 1.27 1.27)) (justify right))
     )
-    (property "Footprint" "LED_SMD:LED_0805_2012Metric" (at 215.9 81.28 0)
+    (property "Footprint" "LED_SMD:LED_0603_1608Metric" (at 215.9 81.28 0)
       (effects (font (size 1.27 1.27)) hide)
     )
@@
       (effects (font (size 1.27 1.27)))
     )
-    (property "Footprint" "Capacitor_SMD:C_0805_2012Metric" (at 261.62 30.7848 0)
+    (property "Footprint" "Capacitor_SMD:C_0603_1608Metric" (at 261.62 30.7848 0)
       (effects (font (size 1.27 1.27)) hide)
     )
@@
       (effects (font (size 1.27 1.27)) (justify left))
     )
-    (property "Footprint" "Resistor_SMD:R_0805_2012Metric" (at 103.632 64.77 90)
+    (property "Footprint" "Resistor_SMD:R_0603_1608Metric" (at 103.632 64.77 90)
       (effects (font (size 1.27 1.27)) hide)
     )
@@
       (effects (font (size 1.27 1.27)) (justify left))
     )
-    (property "Footprint" "Capacitor_Tantalum_SMD:CP_EIA-3216-18_Kemet-A" (at 89.8652 36.83 0)
+    (property "Footprint" "Capacitor_SMD:C_1206_3216Metric" (at 89.8652 36.83 0)
       (effects (font (size 1.27 1.27)) hide)
     )
@@
       (effects (font (size 1.27 1.27)))
     )
-    (property "Footprint" "Capacitor_SMD:C_0805_2012Metric" (at 261.62 43.4848 0)
+    (property "Footprint" "Capacitor_SMD:C_0603_1608Metric" (at 261.62 43.4848 0)
       (effects (font (size 1.27 1.27)) hide)
     )
@@
       (effects (font (size 1.27 1.27)) (justify left))
     )
-    (property "Footprint" "Resistor_SMD:R_0805_2012Metric" (at 188.722 90.17 90)
+    (property "Footprint" "Resistor_SMD:R_0603_1608Metric" (at 188.722 90.17 90)
       (effects (font (size 1.27 1.27)) hide)
     )
@@
       (effects (font (size 1.27 1.27)) (justify left))
     )
-    (property "Footprint" "Resistor_SMD:R_0805_2012Metric" (at 201.422 90.17 90)
+    (property "Footprint" "Resistor_SMD:R_0603_1608Metric" (at 201.422 90.17 90)
       (effects (font (size 1.27 1.27)) hide)
     )
@@
       (effects (font (size 1.27 1.27)) (justify right))
     )
-    (property "Footprint" "LED_SMD:LED_0805_2012Metric" (at 152.4 81.28 0)
+    (property "Footprint" "LED_SMD:LED_0603_1608Metric" (at 152.4 81.28 0)
       (effects (font (size 1.27 1.27)) hide)
     )
@@
       (effects (font (size 1.27 1.27)) (justify left))
     )
-    (property "Footprint" "Capacitor_SMD:C_0805_2012Metric" (at 36.5252 36.83 0)
+    (property "Footprint" "Capacitor_SMD:C_0603_1608Metric" (at 36.5252 36.83 0)
       (effects (font (size 1.27 1.27)) hide)
     )
@@
       (effects (font (size 1.27 1.27)) (justify left))
     )
-    (property "Footprint" "Resistor_SMD:R_0805_2012Metric" (at 150.622 90.17 90)
-      (effects (font (size 1.27 1.27)) hide)
-    )
+    (property "Footprint" "Resistor_SMD:R_0603_1608Metric" (at 150.622 90.17 90)
+      (effects (font (size 1.27 1.27)) hide)
+    )

Commit message: [pcb] Start reworking pcb with 0603 components
Parts:
- FB1: footprint Inductor_SMD:L_0603_1608Metric -> Capacitor_SMD:C_0603_1608Metric
Changed lines of the file:
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@@
       (effects (font (size 1.27 1.27)))
     )
-    (property "Footprint" "Inductor_SMD:L_0603_1608Metric" (at 82.55 29.718 90)
+    (property "Footprint" "Capacitor_SMD:C_0603_1608Metric" (at 82.55 29.718 90)
       (effects (font (size 1.27 1.27)) hide)
     )

Commit message: [pcb] Routing on smaller board. Before removal of button.
Parts:
- removed C17: 100nF, Capacitor_SMD:C_0603_1608Metric, symbol Device:C
- removed R11: 1kR, Resistor_SMD:R_0603_1608Metric, symbol Device:R
- removed R9: 10kR, Resistor_SMD:R_0603_1608Metric, symbol Device:R
- removed SW3: STOP, Autko:12mm_tact_switch, symbol Switch:SW_Push
Connections:
- net BTN_STOP is gone; now on net USR_BTN: U3.11 (PC1)
- net BTN_START renamed USR_BTN
- net USR_BTN: no longer U3.10 (PC0)
- no-connect marks 7 -> 8
Other:
- moved on the sheet: C10, C18, X1
